File: electronics/view_base/view_base.kicad_sch (KiCad schematic)
At the start: 258 parts, among them J1 USB_C_Receptacle_USB2.0, J2 A, J3 B, J4 LCD, J5 59453-081110EDHLF, J6 BLDC, J7 SM04B-SRSS-TB(LF)(SN), J8 SM04B-SRSS-TB(LF)(SN), J9 SM04B-SRSS-TB(LF)(SN), Q1 MMBT4403, Q4 BSS138, Q5 BSS138, SW1 RST, SW2 Boot, U1 SN74LV1T34DBV, U11 ESP32-S3-WROOM-1U-N16R8, U2 MT6701-CT, U3 VEML7700, U4 AMS1117-3.3, U5 USBLC6-2SC6, U6 HX711, U7 VL53L0CXV0DH_1, U8 LP5907MFX-2.8, U8 TMC6300

Commit message: update to kicad 9.0
Parts:
- J5: Mouser 649-59453081110EDHLF -> 649-59453081110EDHLF
- U10: renamed from U8; Mouser 595-LP5907MFX-2.8NPB -> 595-LP5907MFX-2.8NPB
- U9: renamed from U7; Mouser 511-VL53L0CXV0DH/1 -> 511-VL53L0CXV0DH/1
- renumbered C27 to C93, C38 to C94, C39 to C95, Q4 to Q2, Q5 to Q3, R18 to R23, R23 to R24, R22 to R25, R19 to R26, R21 to R27, R20 to R28
